File: eagle/portenta_h7_repin.brd (EAGLE design)
At the start: 66 x 25.4 mm, 5 parts, among them J1 HIROSE_DF40C-80DS-0.4V_51HIRO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, J2 HIROSE_DF40C-80DS-0.4V_51HIRO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

Commit message: fix serial1
Connections:
- net J1-33: now also J1.17; no longer J1.25
- net J1-35: now also J1.18; no longer J1.26
Routing:
- net GND: track 191.6 -> 196.6 mm
- net VIN: track 33.4 -> 36.7 mm
- net 5V: track 20.6 -> 23.5 mm
- net J1-33: track 32.0 -> 34.8 mm
- net J1-35: track 33.1 -> 35.5 mm
Other:
- board text added: "v1.1"
