File: eagle/portenta_h7_repin.sch (EAGLE design)
At the start: 5 parts, among them J1 HIROSE_DF40C-80DS-0.4V_51HIRO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, J2 HIROSE_DF40C-80DS-0.4V_51HIRO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

Commit message: fix serial1
Connections:
- net J1-33: now also J1A.17; no longer J1A.25
- net J1-35: now also J1A.18; no longer J1A.26
Other:
- note added: "v1.1"
- note removed: "v1.0"
Changed lines of the file:
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@@
 <?xml version="1.0" encoding="utf-8"?>
 <!DOCTYPE eagle SYSTEM "eagle.dtd">
-<eagle version="9.2.2">
+<eagle version="9.6.2">
 <drawing>
 <settings>
@@
 gbr1.github.io
 giovannididio.bruno@gmail.com</text>
-<text x="375.92" y="5.08" size="2.54" layer="91">v1.0</text>
+<text x="375.92" y="5.08" size="2.54" layer="91">v1.1</text>
 <text x="345.44" y="20.32" size="2.54" layer="91">GPL v3.0</text>
 </plain>
@@
 </segment>
 <segment>
-<pinref part="J1" gate="A" pin="25"/>
-<wire x1="33.02" y1="116.84" x2="40.64" y2="116.84" width="0.1524" layer="91"/>
-<label x="40.64" y="116.84" size="1.778" layer="95" xref="yes"/>
+<pinref part="J1" gate="A" pin="17"/>
+<wire x1="33.02" y1="157.48" x2="40.64" y2="157.48" width="0.1524" layer="91"/>
+<label x="40.64" y="157.48" size="1.778" layer="95" xref="yes"/>
 </segment>
 </net>
@@
 </segment>
 <segment>
-<pinref part="J1" gate="A" pin="26"/>
-<wire x1="33.02" y1="111.76" x2="40.64" y2="111.76" width="0.1524" layer="91"/>
-<label x="40.64" y="111.76" size="1.778" layer="95" xref="yes"/>
-</segment>
-</net>
+<pinref part="J1" gate="A" pin="18"/>
+<wire x1="33.02" y1="152.4" x2="40.64" y2="152.4" width="0.1524" layer="91"/>
+<label x="40.64" y="152.4" size="1.778" layer="95" xref="yes"/>
+</segment>
+</net>
